File: Matrice LED.kicad_pcb (KiCad board)
At the start: 2 copper layers, 65.6 x 67 mm, 3 parts, among them J1 Conn_01x03_Socket, J2 USB_B

Commit message: New layout
Parts:
- added J3: USB_B, Connector_USB:USB_B_Lumberg_2411_02_Horizontal, F.Cu at (88.5, 33.5)
- added J4: USB_B, Connector_USB:USB_B_Lumberg_2411_02_Horizontal, F.Cu at (35.4, 33.5)
- A1: footprint Module:RaspberryPi_Pico_Common_Unspecified -> PCM_SL_Development_Boards:raspberry_pi_pico_THT; moved to F.Cu
- J2: moved to F.Cu
- moved J2 125.8 mm to (54.0, 35.4), turned to 90 degrees
- moved J1 117.0 mm to (28.4, 55.5), turned to 180 degrees
- moved A1 87.5 mm to (87.0, 45.2), turned to -90 degrees
Routing:
- net unconnected-(A1-GPIO8-Pad11): track 132.4 -> 0.00 mm, vias 2 -> 0
- net GND: track 234.3 -> 130.3 mm, vias 4 -> 0
- net +5V: track 70.1 -> 142.8 mm, vias 1 -> 0
- net /GP4: track 43.6 -> 61.5 mm, vias 2 -> 0
Other:
- board size 65.6 x 67 mm -> 70 x 50 mm

Commit message: Final version
As ordered from PCBWay on 26/03/2026
Parts:
- removed J3, J4: USB_B, Connector_USB:USB_B_Lumberg_2411_02_Horizontal
- added GP0: Push_Button_W12mm, PCM_SL_Footprints:Push_Button_W12mm, F.Cu at (79.0, 30.0)
- J1: footprint Connector_PinSocket_2.54mm:PinSocket_1x03_P2.54mm_Vertical -> Connector_JST:JST_EH_B3B-EH-A_1x03_P2.50mm_Vertical
- moved J1 27.7 mm to (46.5, 34.6), turned to 90 degrees
- moved J2 7.21 mm to (61.2, 35.0)
- moved A1 0.83 mm to (86.2, 45.0)
Connections:
- A1 pad 1: unconnected-(A1-GPIO0-Pad1) -> Net-(A1-GPIO0)
- A1 pad 36: unconnected-(A1-3V3-Pad36) -> Net-(A1-3V3)
- J1 pad 2: /GP4 -> GND
- J1 pad 3: GND -> /GP4
Routing:
- net +5V: track 142.8 -> 57.4 mm
- net Net-(A1-3V3): track 0.00 -> 56.4 mm
- net GND: track 130.3 -> 159.2 mm
- net Net-(A1-GPIO0): track 0.00 -> 26.3 mm
- net /GP4: track 61.5 -> 47.4 mm
Other:
- board size 70 x 50 mm -> 55 x 50 mm
- board text added: "3.3V"
- board text added: "5V"
- board text added: "GP0"
- board text removed: "VCC"
