File: Matrice LED.kicad_sch (KiCad schematic)
At the start: 3 parts, among them J1 Conn_01x03_Socket, J2 USB_B

Commit message: Juste pour voir
Other:
- note added: "Un commentaire"
Changed lines of the file:
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@@
 	(generator_version "9.0")
 	(paper "A4")
+	(text "Un commentaire "
+		(exclude_from_sim no)
+		(at 83.82 112.776 0)
+		(effects
+			(font
+				(size 1.27 1.27)
+			)
+		)
+	)
 	(junction
 		(at 62.23 100.33)

Commit message: Fix #1
Other:
- note removed: "Un commentaire"
Changed lines of the file:
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@@
 	(generator_version "9.0")
 	(paper "A4")
-	(text "Un commentaire "
-		(exclude_from_sim no)
-		(at 83.82 112.776 0)
-		(effects
-			(font
-				(size 1.27 1.27)
-			)
-		)
-	)
 	(junction
 		(at 62.23 100.33)

Commit message: New layout
Parts:
- added J3, J4: USB_B, Connector_USB:USB_B_Lumberg_2411_02_Horizontal, symbol Connector:USB_B
Connections:
- net +5V: now also J3.1 (VBUS), J4.1 (VBUS)
- net GND: now also J3.4 (GND), J3.5 (Shield), J4.4 (GND), J4.5 (Shield)
- no-connect marks 0 -> 6

Commit message: Final version
As ordered from PCBWay on 26/03/2026
Parts:
- removed J3, J4: USB_B, Connector_USB:USB_B_Lumberg_2411_02_Horizontal, symbol Connector:USB_B
- added SW1: Push_Button_W12mm, PCM_SL_Footprints:Push_Button_W12mm, symbol PCM_SL_Devices:Push_Button_W12mm
- J1: footprint Connector_PinSocket_2.54mm:PinSocket_1x03_P2.54mm_Vertical -> Connector_JST:JST_EH_B3B-EH-A_1x03_P2.50mm_Vertical; symbol Connector:Conn_01x03_Socket -> PCM_SL_Connectors:JST_03
Connections:
- net GND: now also J1.2; no longer J1.3 (Pin_3)
- net GP4: now also J1.3; no longer J1.2 (Pin_2)
- net at A1.1 (GPIO0): now also SW1.2
- net at A1.36 (3V3): now also SW1.1
- no-connect marks 6 -> 2
